File: TcBox_6x4.kicad_pcb (KiCad board)
At the start: 2 copper layers, 42.7 x 73.7 mm, 13 parts, among them J1 Conn_01x25, J2 Conn_01x06_Male, J3 Conn_01x06_Male, J4 Conn_01x06_Male, J5 Conn_01x06_Male

Commit message: First draft. Going to branch here and try a different footprint option.
Parts:
- added R1: DNF (short), coldMount_footprints_src:thruVia, F.Cu at (150.8, 60.2)
Routing:
- net /Ch3_1: track 61.9 -> 61.4 mm
- net /coldMount: vias 0 -> 53
- added copper zone on B.Cu, net /coldMount
- added copper zone on F.Cu, net /coldMount
Other:
- outline, holes or cut-outs redrawn
- board text removed: "J2"
- board text removed: "J3"

Commit message: Generated gerbers
Parts:
- J2, J3, J4, J5: footprint coldMount_footprints_src:WB_pad_6ch -> coldMount_footprints_src:WB_pad_6ch_thickStacked
- moved J3 1.05 mm to (135.9, 117.5)
- moved J2 0.60 mm to (135.9, 108.0)
- moved J4 0.33 mm to (165.4, 118.5)
- moved J5 0.33 mm to (165.4, 108.5)
Connections:
- J2 pad 2: /Ch0_1 -> /Ch0_2
- J2 pad 3: /Ch0_2 -> /Ch0_4
- J2 pad 4: /Ch0_3 -> /Ch0_1
- J2 pad 5: /Ch0_4 -> /Ch0_3
- J3 pad 2: /Ch1_1 -> /Ch1_2
- J3 pad 3: /Ch1_2 -> /Ch1_4
- J3 pad 4: /Ch1_3 -> /Ch1_1
- J3 pad 5: /Ch1_4 -> /Ch1_3
- J4 pad 2: /Ch2_1 -> /Ch2_2
- J4 pad 3: /Ch2_2 -> /Ch2_4
- J4 pad 4: /Ch2_3 -> /Ch2_1
- J4 pad 5: /Ch2_4 -> /Ch2_3
- J5 pad 2: /Ch3_1 -> /Ch3_2
- J5 pad 3: /Ch3_2 -> /Ch3_4
- J5 pad 4: /Ch3_3 -> /Ch3_1
- J5 pad 5: /Ch3_4 -> /Ch3_3
Routing:
- net /Ch3_2: track 62.3 -> 64.4 mm
- net /Ch0_1: track 59.3 -> 61.2 mm
- net /Ch0_5: track 66.4 -> 68.2 mm
- net /Ch3_5: track 56.8 -> 58.3 mm
- net /Ch2_5: track 66.4 -> 67.9 mm
- net /Ch0_3: track 62.2 -> 63.5 mm
- net /Ch3_3: track 58.9 -> 60.2 mm
- net /Ch2_3: track 69.7 -> 71.0 mm
- net /Ch1_1: track 70.4 -> 71.7 mm
- net /Ch3_1: track 61.4 -> 62.6 mm
- net /Ch1_3: track 73.8 -> 74.9 mm
- net /Ch2_1: track 73.0 -> 74.2 mm
- net /Ch1_5: track 78.8 -> 79.7 mm
- net /Ch2_0: track 78.8 -> 78.0 mm
- net /Ch1_4: track 73.0 -> 72.3 mm
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