File: TcBox_6x4.kicad_sch (KiCad schematic)
At the start: 13 parts, among them J1 Conn_01x25, J2 Conn_01x06_Male, J3 Conn_01x06_Male, J4 Conn_01x06_Male, J5 Conn_01x06_Male

Commit message: First draft. Going to branch here and try a different footprint option.
Parts:
- added R1: DNF (short), coldMount_footprints_src:thruVia, symbol Device:R
Connections:
- new net coldMount: R1.1, R1.2
Changed lines of the file:
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@@
+    (stroke (width 0) (type default) (color 0 0 0 0))
+  )
+  (wire (pts (xy 110.49 41.91) (xy 110.49 45.72))
     (stroke (width 0) (type default) (color 0 0 0 0))
   )
@@
     (stroke (width 0) (type default) (color 0 0 0 0))
   )
+  (wire (pts (xy 110.49 31.75) (xy 110.49 34.29))
+    (stroke (width 0) (type default) (color 0 0 0 0))
+  )
   (wire (pts (xy 67.31 101.6) (xy 69.85 101.6))
     (stroke (width 0) (type default) (color 0 0 0 0))
@@
     (effects (font (size 1.27 1.27)) (justify right bottom))
   )
+  (label "coldMount" (at 110.49 31.75 0)
+    (effects (font (size 1.27 1.27)) (justify left bottom))
+  )
   (label "Ch2_4" (at 69.85 111.76 0)
     (effects (font (size 1.27 1.27)) (justify left bottom))
@@
   (label "Ch0_1" (at 64.77 57.15 180)
     (effects (font (size 1.27 1.27)) (justify right bottom))
+  )
+  (label "coldMount" (at 110.49 45.72 0)
+    (effects (font (size 1.27 1.27)) (justify left bottom))
   )
   (label "Ch2_1" (at 64.77 41.91 180)
@@
     (pin "5")
     (pin "6")
+  )
+  (symbol (lib_id "Device:R") (at 110.49 38.1 0) (unit 1)
+    (in_bom yes) (on_board yes) (fields_autoplaced)
+    (property "Reference" "R1" (id 0) (at 112.268 37.2653 0)
+      (effects (font (size 1.27 1.27)) (justify left))
+    )
+    (property "Value" "DNF (short)" (id 1) (at 112.268 39.8022 0)
+      (effects (font (size 1.27 1.27)) (justify left))
+    )
+    (property "Footprint" "coldMount_footprints_src:thruVia" (id 2) (at 108.712 38.1 90)
+      (effects (font (size 1.27 1.27)) hide)
+    )
+    (property "Datasheet" "~" (id 3) (at 110.49 38.1 0)
+      (effects (font (size 1.27 1.27)) hide)
+    )
+    (pin "1")
+    (pin "2")
   )
   (symbol (lib_id "Mechanical:MountingHole") (at 25.4 55.88 0) (unit 1)
@@
       (reference "J5") (unit 1) (value "Conn_01x06_Male") (footprint "coldMount_footprints_src:WB_pad_6ch")
     )
-  )
+    (path "/47775f86-7fcd-466d-9ea5-8743bfa7e779"
+      (reference "R1") (unit 1) (value "DNF (short)") (footprint "coldMount_footprints_src:thruVia")
+    )
+  )

Commit message: Generated gerbers
Parts:
- J2, J3, J4, J5: footprint coldMount_footprints_src:WB_pad_6ch -> coldMount_footprints_src:WB_pad_6ch_thickStacked
Connections:
- net Ch0_1: now also J2.4 (Pin_4); no longer J2.2 (Pin_2)
- net Ch0_2: now also J2.2 (Pin_2); no longer J2.3 (Pin_3)
- net Ch0_3: now also J2.5 (Pin_5); no longer J2.4 (Pin_4)
- net Ch0_4: now also J2.3 (Pin_3); no longer J2.5 (Pin_5)
- net Ch1_1: now also J3.4 (Pin_4); no longer J3.2 (Pin_2)
- net Ch1_2: now also J3.2 (Pin_2); no longer J3.3 (Pin_3)
- net Ch1_3: now also J3.5 (Pin_5); no longer J3.4 (Pin_4)
- net Ch1_4: now also J3.3 (Pin_3); no longer J3.5 (Pin_5)
- net Ch2_1: now also J4.4 (Pin_4); no longer J4.2 (Pin_2)
- net Ch2_2: now also J4.2 (Pin_2); no longer J4.3 (Pin_3)
- net Ch2_3: now also J4.5 (Pin_5); no longer J4.4 (Pin_4)
- net Ch2_4: now also J4.3 (Pin_3); no longer J4.5 (Pin_5)
- net Ch3_1: now also J5.4 (Pin_4); no longer J5.2 (Pin_2)
- net Ch3_2: now also J5.2 (Pin_2); no longer J5.3 (Pin_3)
- net Ch3_3: now also J5.5 (Pin_5); no longer J5.4 (Pin_4)
- net Ch3_4: now also J5.3 (Pin_3); no longer J5.5 (Pin_5)
Changed lines of the file:
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@@
     (stroke (width 0) (type default) (color 0 0 0 0))
   )
-  (label "Ch1_1" (at 52.07 104.14 0)
+  (label "Ch1_1" (at 52.07 109.22 0)
     (effects (font (size 1.27 1.27)) (justify left bottom))
   )
@@
     (effects (font (size 1.27 1.27)) (justify right bottom))
   )
-  (label "Ch1_4" (at 52.07 111.76 0)
+  (label "Ch1_4" (at 52.07 106.68 0)
     (effects (font (size 1.27 1.27)) (justify left bottom))
   )
@@
     (effects (font (size 1.27 1.27)) (justify left bottom))
   )
-  (label "Ch0_2" (at 35.56 106.68 0)
+  (label "Ch0_2" (at 35.56 104.14 0)
     (effects (font (size 1.27 1.27)) (justify left bottom))
   )
@@
     (effects (font (size 1.27 1.27)) (justify right bottom))
   )
-  (label "Ch2_2" (at 69.85 106.68 0)
+  (label "Ch2_2" (at 69.85 104.14 0)
     (effects (font (size 1.27 1.27)) (justify left bottom))
   )
@@
     (effects (font (size 1.27 1.27)) (justify left bottom))
   )
-  (label "Ch1_2" (at 52.07 106.68 0)
+  (label "Ch1_2" (at 52.07 104.14 0)
     (effects (font (size 1.27 1.27)) (justify left bottom))
   )
@@
     (effects (font (size 1.27 1.27)) (justify right bottom))
   )
-  (label "Ch3_4" (at 87.63 111.76 0)
+  (label "Ch3_4" (at 87.63 106.68 0)
     (effects (font (size 1.27 1.27)) (justify left bottom))
   )
@@
     (effects (font (size 1.27 1.27)) (justify left bottom))
   )
-  (label "Ch2_1" (at 69.85 104.14 0)
+  (label "Ch2_1" (at 69.85 109.22 0)
     (effects (font (size 1.27 1.27)) (justify left bottom))
   )
@@
     (effects (font (size 1.27 1.27)) (justify left bottom))
   )
-  (label "Ch2_4" (at 69.85 111.76 0)
-    (effects (font (size 1.27 1.27)) (justify left bottom))
-  )
-  (label "Ch2_3" (at 69.85 109.22 0)
-    (effects (font (size 1.27 1.27)) (justify left bottom))
-  )
-  (label "Ch0_1" (at 35.56 104.14 0)
-    (effects (font (size 1.27 1.27)) (justify left bottom))
-  )
-  (label "Ch3_1" (at 87.63 104.14 0)
+  (label "Ch2_4" (at 69.85 106.68 0)
+    (effects (font (size 1.27 1.27)) (justify left bottom))
+  )
+  (label "Ch2_3" (at 69.85 111.76 0)
+    (effects (font (size 1.27 1.27)) (justify left bottom))
+  )
+  (label "Ch0_1" (at 35.56 109.22 0)
+    (effects (font (size 1.27 1.27)) (justify left bottom))
+  )
+  (label "Ch3_1" (at 87.63 109.22 0)
     (effects (font (size 1.27 1.27)) (justify left bottom))
   )
@@
     (effects (font (size 1.27 1.27)) (justify right bottom))
   )
-  (label "Ch1_3" (at 52.07 109.22 0)
-    (effects (font (size 1.27 1.27)) (justify left bottom))
-  )
-  (label "Ch0_3" (at 35.56 109.22 0)
+  (label "Ch1_3" (at 52.07 111.76 0)
+    (effects (font (size 1.27 1.27)) (justify left bottom))
+  )
+  (label "Ch0_3" (at 35.56 111.76 0)
     (effects (font (size 1.27 1.27)) (justify left bottom))
   )
@@
     (effects (font (size 1.27 1.27)) (justify left bottom))
   )
-  (label "Ch3_3" (at 87.63 109.22 0)
+  (label "Ch3_3" (at 87.63 111.76 0)
     (effects (font (size 1.27 1.27)) (justify left bottom))
   )
@@
     (effects (font (size 1.27 1.27)) (justify right bottom))
   )
-  (label "Ch0_4" (at 35.56 111.76 0)
+  (label "Ch0_4" (at 35.56 106.68 0)
     (effects (font (size 1.27 1.27)) (justify left bottom))
   )
@@
     (effects (font (size 1.27 1.27)) (justify right bottom))
   )
-  (label "Ch3_2" (at 87.63 106.68 0)
+  (label "Ch3_2" (at 87.63 104.14 0)
     (effects (font (size 1.27 1.27)) (justify left bottom))
   )
@@
     (property "Reference" "J4" (id 0) (at 68.58 97.79 0))
     (property "Value" "Conn_01x06_Male" (id 1) (at 68.58 118.11 0))
-    (property "Footprint" "coldMount_footprints_src:WB_pad_6ch" (id 2) (at 62.23 106.68 0)
+    (property "Footprint" "coldMount_footprints_src:WB_pad_6ch_thickStacked" (id 2) (at 62.23 106.68 0)
       (effects (font (size 1.27 1.27)) hide)
     )
@@
     (property "Reference" "J5" (id 0) (at 86.36 97.79 0))
     (property "Value" "Conn_01x06_Male" (id 1) (at 87.63 118.11 0))
-    (property "Footprint" "coldMount_footprints_src:WB_pad_6ch" (id 2) (at 80.01 106.68 0)
+    (property "Footprint" "coldMount_footprints_src:WB_pad_6ch_thickStacked" (id 2) (at 80.01 106.68 0)
       (effects (font (size 1.27 1.27)) hide)
     )
@@
     (property "Reference" "J2" (id 0) (at 34.29 97.79 0))
     (property "Value" "Conn_01x06_Male" (id 1) (at 30.48 118.11 0))
-    (property "Footprint" "coldMount_footprints_src:WB_pad_6ch" (id 2) (at 27.94 106.68 0)
+    (property "Footprint" "coldMount_footprints_src:WB_pad_6ch_thickStacked" (id 2) (at 27.94 106.68 0)
       (effects (font (size 1.27 1.27)) hide)
     )
@@
     (property "Reference" "J3" (id 0) (at 50.8 97.79 0))
     (property "Value" "Conn_01x06_Male" (id 1) (at 49.53 118.11 0))
-    (property "Footprint" "coldMount_footprints_src:WB_pad_6ch" (id 2) (at 44.45 106.68 0)
+    (property "Footprint" "coldMount_footprints_src:WB_pad_6ch_thickStacked" (id 2) (at 44.45 106.68 0)
       (effects (font (size 1.27 1.27)) hide)
     )
@@
     )
     (path "/96bccfc7-b5ef-4d0c-a365-c58ad6131ed3"
-      (reference "J2") (unit 1) (value "Conn_01x06_Male") (footprint "coldMount_footprints_src:WB_pad_6ch")
+      (reference "J2") (unit 1) (value "Conn_01x06_Male") (footprint "coldMount_footprints_src:WB_pad_6ch_thickStacked")
     )
     (path "/f201fa02-1ff4-4a2e-a833-aec3fb121c91"
-      (reference "J3") (unit 1) (value "Conn_01x06_Male") (footprint "coldMount_footprints_src:WB_pad_6ch")
+      (reference "J3") (unit 1) (value "Conn_01x06_Male") (footprint "coldMount_footprints_src:WB_pad_6ch_thickStacked")
     )
     (path "/130dbdd0-cc0b-4640-99bc-a97cf806451d"
-      (reference "J4") (unit 1) (value "Conn_01x06_Male") (footprint "coldMount_footprints_src:WB_pad_6ch")
+      (reference "J4") (unit 1) (value "Conn_01x06_Male") (footprint "coldMount_footprints_src:WB_pad_6ch_thickStacked")
     )
     (path "/279867f8-840d-401b-9e06-8673d94bed4c"
-      (reference "J5") (unit 1) (value "Conn_01x06_Male") (footprint "coldMount_footprints_src:WB_pad_6ch")
+      (reference "J5") (unit 1) (value "Conn_01x06_Male") (footprint "coldMount_footprints_src:WB_pad_6ch_thickStacked")
     )
     (path "/47775f86-7fcd-466d-9ea5-8743bfa7e779"
